File: design/flash_programmer.kicad_pcb (KiCad board)
At the start: 2 copper layers, 61 x 38.1 mm, 49 parts, among them P201 USB_B, P601 ISP, Q301 2N3904, Q701 2N3906, U201 FT230X, U301 GLS27SF010, U401 MAX662A, U501 74HC595, U502 74HC595, U601 ATMEGA328P

Commit message: Correction: ATMEGA328P -> ATMEGA328-AU
Parts:
- U601: value ATMEGA328P -> ATMEGA328-AU
Changed lines of the file:
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@@
       (effects (font (size 0.65 0.65) (thickness 0.15)))
     )
-    (fp_text value ATMEGA328P (at 0 0 180) (layer F.Fab)
+    (fp_text value ATMEGA328-AU (at 0 0 180) (layer F.Fab)
       (effects (font (size 0.65 0.65) (thickness 0.15)))
     )

Commit message: Add license and OSHW logo to PCB
Parts:
- removed G***: LOGO, logo:logo
- added REF***: OSHW-Logo2_14.6x12mm_SilkScreen, Symbols:OSHW-Logo2_14.6x12mm_SilkScreen, B.Cu at (49.5, 54.6)
Other:
- board text added: "Copyright 2017 John DiSanti"
- board text added: "Copyright 2017 John DiSanti Copyright and related rights are licensed under the Solderpad Hardware License, Version 0.51 (the "License"); you may not use this document except in compliance with the License. You may obtain a copy of the License at http://solderpad.org/licenses/SHL-0.51. Unless required by applicable law or agreed to in writing, software, hardware and materials distributed under th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"
- board text removed: "John DiSanti"
- board text removed: "March 12, 2017"

Commit message: Add PDFs of schematic and PCB, and add BOM file
Other:
- board text added: "Copyright and related rights are licensed under the Solderpad Hardware License, Version 0.51 (the "License"); you may not use this document except in compliance with the License. You may obtain a copy of the License at http://solderpad.org/licenses/SHL-0.51. Unless required by applicable law or agreed to in writing, software, hardware and materials distributed under this License is distributed on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"
- board text removed: "Copyright 2017 John DiSanti Copyright and related rights are licensed under the Solderpad Hardware License, Version 0.51 (the "License"); you may not use this document except in compliance with the License. You may obtain a copy of the License at http://solderpad.org/licenses/SHL-0.51. Unless required by applicable law or agreed to in writing, software, hardware and materials distributed under th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"
Changed lines of the file:
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@@
 (kicad_pcb (version 4) (host pcbnew 4.0.5)
   (general
-    (links 0)
+    (links 141)
     (no_connects 0)
-    (area 38.049999 38.049999 99.110001 76.250001)
+    (area 20.32 32.86 151.462859 196.955)
     (thickness 1.6)
     (drawings 59)
@@
     (nets 73)
   )
-  (page A4)
+  (page USLetter)
+  (title_block
+    (title "GLS27SF010 Flash Programmer")
+    (date 2017-05-06)
+    (company "Copyright 2017 John DiSanti")
+  )
   (layers
     (0 F.Cu signal)
@@
     (visible_elements 7FFFFFFF)
     (pcbplotparams
-      (layerselection 0x10000_00000000)
+      (layerselection 0x01100_00000001)
       (usegerberextensions false)
       (excludeedgelayer true)
@@
       (hpglpenoverlay 2)
       (psnegative false)
-      (psa4output true)
+      (psa4output false)
       (plotreference false)
       (plotvalue true)
@@
       (padsonsilk false)
       (subtractmaskfromsilk false)
-      (outputformat 2)
-      (mirror true)
+      (outputformat 4)
+      (mirror false)
       (drillshape 0)
       (scaleselection 1)
@@
       (xy -0.026262 5.547126) (xy 0 5.547126) (xy 0.209014 5.547002)) (layer B.SilkS) (width 0.01))
   )
-  (gr_text "Copyright 2017 John DiSanti\n\nCopyright and related rights are licensed under the Solderpad Hardware License, Version 0.51 (the \"License\");\nyou may not use this document except in compliance with the License. You may obtain a copy of the License at\nhttp://solderpad.org/licenses/SHL-0.51. Unless required by applicable law or agreed to in writing, software,\nhardware and materials distributed under this License is distributed on an \"AS IS\" BASIS, WITHOUT WARRANTIES\nOR CONDITIONS OF ANY KIND, either express or implied. See the License for the specific language governing\npermissions and limitations under the License." (at 25.4 180.34) (layer Dwgs.User)
+  (gr_text "Copyright and related rights are licensed under the Solderpad Hardware License, Version 0.51 (the \"License\");\nyou may not use this document except in compliance with the License. You may obtain a copy of the License at\nhttp://solderpad.org/licenses/SHL-0.51. Unless required by applicable law or agreed to in writing, software,\nhardware and materials distributed under this License is distributed on an \"AS IS\" BASIS, WITHOUT WARRANTIES\nOR CONDITIONS OF ANY KIND, either express or implied. See the License for the specific language governing\npermissions and limitations under the License." (at 20.32 189.23) (layer Dwgs.User)
     (effects (font (size 1.5 1.5) (thickness 0.3)) (justify left))
   )
